Commit message: Inertia Added

File: gaz_sim/quad_description.xacro (robot description, xacro)
@@ -41,4 +41,8 @@
 <material name = "orange"/>
 </visual>
+<inertial>
+    <mass value = "1"/>
+    <inertia ixx="0.02604167" ixy="0.0" ixz="0.0" iyy="0.088541" iyz="0.0" izx="0.0" izy="0.0" izz=".1041667"/>
+ </inertial>
 </link>
 <!--upper left limb-->
@@ -57,4 +61,8 @@
 <material name = "red"/>
 </visual>
+<inertial>
+    <mass value= "0.25"/>
+    <inertia ixx="0.005364" ixy="0.0" ixz="0.0" iyy="0.005364" iyz="0.0" izx="0.0" izy="0.0" izz="0.0003125"/>
+ </inertial>
 </link>
 <link name = "ulf_leg">
@@ -103,4 +111,8 @@
 <material name = "red"/>
 </visual>
+<inertial>
+    <mass value= "0.25"/>
+    <inertia ixx="0.005364" ixy="0.0" ixz="0.0" iyy="0.005364" iyz="0.0" izx="0.0" izy="0.0" izz="0.0003125"/>
+ </inertial>
 </link>
 <link name = "urf_leg">
@@ -149,4 +161,8 @@
 <material name = "red"/>
 </visual>
+<inertial>
+    <mass value= "0.25"/>
+    <inertia ixx="0.005364" ixy="0.0" ixz="0.0" iyy="0.005364" iyz="0.0" izx="0.0" izy="0.0" izz="0.0003125"/>
+ </inertial>
 </link>
 <link name = "blf_leg">
@@ -195,4 +211,8 @@
 <material name = "red"/>
 </visual>
+<inertial>
+    <mass value= "0.25"/>
+    <inertia ixx="0.005364" ixy="0.0" ixz="0.0" iyy="0.005364" iyz="0.0" izx="0.0" izy="0.0" izz="0.0003125"/>
+ </inertial>
 </link>
 <link name = "brf_leg">

Commit message: Femur joint added, Constraints left

File: gaz_sim/quad_description.xacro (robot description, xacro)
@@ -81,4 +81,19 @@
   </visual>
 </link>
+<link name = "ulf_femur">
+  <pose>0 0 0 0 0 0</pose>
+  <collision name = "collision_ulf_femur">
+    <geometry>
+      <cylinder length = "0.5" radius = "0.05"/>
+    </geometry>
+  </collision>
+  <visual>
+    <origin rpy = "0 0 0" xyz = "0 0 0"/>
+    <geometry>
+      <cylinder length = "0.5" radius = "0.05"/>
+    </geometry>
+    <material name = "brown" />
+  </visual>
+</link>
 <link name = "ulf_paw">
   <pose>0 0 0 0 0 0</pose>
@@ -131,4 +146,19 @@
   </visual>
 </link>
+<link name = "urf_femur">
+  <pose>0 0 0 0 0 0</pose>
+  <collision name = "collision_urf_femur">
+    <geometry>
+      <cylinder length = "0.5" radius = "0.05"/>
+    </geometry>
+  </collision>
+  <visual>
+    <origin rpy = "0 0 0" xyz = "0 0 0"/>
+    <geometry>
+      <cylinder length = "0.5" radius = "0.05"/>
+    </geometry>
+    <material name = "brown" />
+  </visual>
+</link>
 <link name = "urf_paw">
   <pose>0 0 0 0 0 0</pose>
@@ -181,4 +211,19 @@
   </visual>
 </link>
+<link name = "blf_femur">
+  <pose>0 0 0 0 0 0</pose>
+  <collision name = "collision_blf_femur">
+    <geometry>
+      <cylinder length = "0.5" radius = "0.05"/>
+    </geometry>
+  </collision>
+  <visual>
+    <origin rpy = "0 0 0" xyz = "0 0 0"/>
+    <geometry>
+      <cylinder length = "0.5" radius = "0.05"/>
+    </geometry>
+    <material name = "brown" />
+  </visual>
+</link>
 <link name = "blf_paw">
   <pose>0 0 0 0 0 0</pose>
@@ -231,4 +276,19 @@
   </visual>
 </link>
+<link name = "brf_femur">
+  <pose>0 0 0 0 0 0</pose>
+  <collision name = "collision_brf_femur">
+    <geometry>
+      <cylinder length = "0.5" radius = "0.05"/>
+    </geometry>
+  </collision>
+  <visual>
+    <origin rpy = "0 0 0" xyz = "0 0 0"/>
+    <geometry>
+      <cylinder length = "0.5" radius = "0.05"/>
+    </geometry>
+    <material name = "brown" />
+  </visual>
+</link>
 <link name = "brf_paw">
   <pose>0 0 0 0 0 0</pose>
@@ -257,13 +317,20 @@
 <joint name = "ulf_2" type = "revolute">
   <parent link = "ulf_limb"/>
+  <child link = "ulf_femur"/>
+    <origin xyz = "0 0 0.25" rpy = "0 1.57 0"/>
+      <limit lower = "-0.785" upper = "0.785" effort = "10" velocity = "3"/>
+      <axis xyz = "0 1 0"/>
+</joint>
+<joint name = "ulf_3" type = "revolute">
+  <parent link = "ulf_femur"/>
   <child link = "ulf_leg"/>
-    <origin xyz = "0 0 0.25" rpy = "0 1.57 0"/>
-      <limit lower = "-0.785" upper = "0.785" effort = "10" velocity = "3"/>
-      <axis xyz = "0 1 0"/>
-</joint>
-<joint name = "ulf_3" type = "fixed">
+    <origin xyz = "0 0 -0.25" rpy = "0 1.57 0"/>
+      <limit lower = "-0.785" upper = "0.785" effort = "10" velocity = "3"/>
+      <axis xyz = "0 1 0"/>
+</joint>
+<joint name = "ulf_4" type = "fixed">
   <parent link = "ulf_leg"/>
   <child link = "ulf_paw"/>
-    <origin xyz = "0 0 0.25" rpy = "0 0 0"/>
+    <origin xyz = "0 0 -0.25" rpy = "0 0 0"/>
 </joint>
 <!--joints for urf-->
@@ -277,13 +344,20 @@
 <joint name = "urf_2" type = "revolute">
   <parent link = "urf_limb"/>
+  <child link = "urf_femur"/>
+    <origin xyz = "0 0 0.25" rpy = "0 1.57 0"/>
+      <limit lower = "-0.785" upper = "0.785" effort = "10" velocity = "3"/>
+      <axis xyz = "0 1 0"/>
+</joint>
+<joint name = "urf_3" type = "revolute">
+  <parent link = "urf_femur"/>
   <child link = "urf_leg"/>
-    <origin xyz = "0 0 0.25" rpy = "0 1.57 0"/>
-      <limit lower = "-0.785" upper = "0.785" effort = "10" velocity = "3"/>
-      <axis xyz = "0 1 0"/>
-</joint>
-<joint name = "urf_3" type = "fixed">
+    <origin xyz = "0 0 -0.25" rpy = "0 1.57 0"/>
+      <limit lower = "-0.785" upper = "0.785" effort = "10" velocity = "3"/>
+      <axis xyz = "0 1 0"/>
+</joint>
+<joint name = "urf_4" type = "fixed">
   <parent link = "urf_leg"/>
   <child link = "urf_paw"/>
-    <origin xyz = "0 0 0.25" rpy = "0 0 0"/>
+    <origin xyz = "0 0 -0.25" rpy = "0 0 0"/>
 </joint>
 <!--joints for blf-->
@@ -297,13 +371,20 @@
 <joint name = "blf_2" type = "revolute">
   <parent link = "blf_limb"/>
+  <child link = "blf_femur"/>
+    <origin xyz = "0 0 0.25" rpy = "0 1.57 0"/>
+      <limit lower = "-0.785" upper = "0.785" effort = "10" velocity = "3"/>
+      <axis xyz = "0 1 0"/>
+</joint>
+<joint name = "blf_3" type = "revolute">
+  <parent link = "blf_femur"/>
   <child link = "blf_leg"/>
-    <origin xyz = "0 0 0.25" rpy = "0 1.57 0"/>
-      <limit lower = "-0.785" upper = "0.785" effort = "10" velocity = "3"/>
-      <axis xyz = "0 1 0"/>
-</joint>
-<joint name = "blf_3" type = "fixed">
+    <origin xyz = "0 0 -0.25" rpy = "0 1.57 0"/>
+      <limit lower = "-0.785" upper = "0.785" effort = "10" velocity = "3"/>
+      <axis xyz = "0 1 0"/>
+</joint>
+<joint name = "blf_4" type = "fixed">
   <parent link = "blf_leg"/>
   <child link = "blf_paw"/>
-    <origin xyz = "0 0 0.25" rpy = "0 0 0"/>
+    <origin xyz = "0 0 -0.25" rpy = "0 0 0"/>
 </joint>
 <!--joints for brf-->
@@ -317,13 +398,20 @@
 <joint name = "brf_2" type = "revolute">
   <parent link = "brf_limb"/>
+  <child link = "brf_femur"/>
+    <origin xyz = "0 0 0.25" rpy = "0 1.57 0"/>
+      <limit lower = "-0.785" upper = "0.785" effort = "10" velocity = "3"/>
+      <axis xyz = "0 1 0"/>
+</joint>
+<joint name = "brf_3" type = "revolute">
+  <parent link = "brf_femur"/>
   <child link = "brf_leg"/>
-    <origin xyz = "0 0 0.25" rpy = "0 1.57 0"/>
-      <limit lower = "-0.785" upper = "0.785" effort = "10" velocity = "3"/>
-      <axis xyz = "0 1 0"/>
-</joint>
-<joint name = "brf_3" type = "fixed">
+    <origin xyz = "0 0 -0.25" rpy = "0 1.57 0"/>
+      <limit lower = "-0.785" upper = "0.785" effort = "10" velocity = "3"/>
+      <axis xyz = "0 1 0"/>
+</joint>
+<joint name = "brf_4" type = "fixed">
   <parent link = "brf_leg"/>
   <child link = "brf_paw"/>
-    <origin xyz = "0 0 0.25" rpy = "0 0 0"/>
+    <origin xyz = "0 0 -0.25" rpy = "0 0 0"/>
 </joint>
 </robot>

Commit message: Constraints added, dimensions and pose altered

File: gaz_sim/quad_description.xacro (robot description, xacro)
@@ -70,11 +70,11 @@
   <collision name = "collision_ulf_leg">
     <geometry>
-      <cylinder length = "0.5" radius = "0.05"/>
-    </geometry>
-  </collision>
-  <visual>
-    <origin rpy = "0 0 0" xyz = "0 0 0"/>
-    <geometry>
-      <cylinder length = "0.5" radius = "0.05"/>
+      <cylinder length = "1.0" radius = "0.05"/>
+    </geometry>
+  </collision>
+  <visual>
+    <origin rpy = "0 0 0" xyz = "0 0 0"/>
+    <geometry>
+      <cylinder length = "1.0" radius = "0.05"/>
     </geometry>
     <material name = "green" />
@@ -135,11 +135,11 @@
   <collision name = "collision_urf_leg">
     <geometry>
-      <cylinder length = "0.5" radius = "0.05"/>
-    </geometry>
-  </collision>
-  <visual>
-    <origin rpy = "0 0 0" xyz = "0 0 0"/>
-    <geometry>
-      <cylinder length = "0.5" radius = "0.05"/>
+      <cylinder length = "1.0" radius = "0.05"/>
+    </geometry>
+  </collision>
+  <visual>
+    <origin rpy = "0 0 0" xyz = "0 0 0"/>
+    <geometry>
+      <cylinder length = "1.0" radius = "0.05"/>
     </geometry>
     <material name = "green" />
@@ -200,11 +200,11 @@
   <collision name = "collision_blf_leg">
     <geometry>
-      <cylinder length = "0.5" radius = "0.05"/>
-    </geometry>
-  </collision>
-  <visual>
-    <origin rpy = "0 0 0" xyz = "0 0 0"/>
-    <geometry>
-      <cylinder length = "0.5" radius = "0.05"/>
+      <cylinder length = "1.0" radius = "0.05"/>
+    </geometry>
+  </collision>
+  <visual>
+    <origin rpy = "0 0 0" xyz = "0 0 0"/>
+    <geometry>
+      <cylinder length = "1.0" radius = "0.05"/>
     </geometry>
     <material name = "green" />
@@ -265,11 +265,11 @@
   <collision name = "collision_brf_leg">
     <geometry>
-      <cylinder length = "0.5" radius = "0.05"/>
-    </geometry>
-  </collision>
-  <visual>
-    <origin rpy = "0 0 0" xyz = "0 0 0"/>
-    <geometry>
-      <cylinder length = "0.5" radius = "0.05"/>
+      <cylinder length = "1.0" radius = "0.05"/>
+    </geometry>
+  </collision>
+  <visual>
+    <origin rpy = "0 0 0" xyz = "0 0 0"/>
+    <geometry>
+      <cylinder length = "1.0" radius = "0.05"/>
     </geometry>
     <material name = "green" />
@@ -311,6 +311,6 @@
   <parent link = "link_chassis"/>
   <child link = "ulf_limb"/>
-    <origin xyz = "0.5 0.25 0" rpy = "0 1.57 0.785"/>
-      <limit lower = "-0.785" upper = "0.785" effort = "10" velocity = "3"/>
+    <origin xyz = "0.5 0.25 -0.1" rpy = "0 1.57 0.785"/>
+      <limit lower = "-1.57" upper = "1.57" effort = "10" velocity = "3"/>
       <axis xyz = "1 0 0"/>
 </joint>
@@ -318,5 +318,5 @@
   <parent link = "ulf_limb"/>
   <child link = "ulf_femur"/>
-    <origin xyz = "0 0 0.25" rpy = "0 1.57 0"/>
+    <origin xyz = "0 0 0.25" rpy = "0 2.355 0"/>
       <limit lower = "-0.785" upper = "0.785" effort = "10" velocity = "3"/>
       <axis xyz = "0 1 0"/>
@@ -325,5 +325,5 @@
   <parent link = "ulf_femur"/>
   <child link = "ulf_leg"/>
-    <origin xyz = "0 0 -0.25" rpy = "0 1.57 0"/>
+    <origin xyz = "0 0 -0.25" rpy = "0 2.355 0"/>
       <limit lower = "-0.785" upper = "0.785" effort = "10" velocity = "3"/>
       <axis xyz = "0 1 0"/>
@@ -332,5 +332,5 @@
   <parent link = "ulf_leg"/>
   <child link = "ulf_paw"/>
-    <origin xyz = "0 0 -0.25" rpy = "0 0 0"/>
+    <origin xyz = "0 0 -0.5" rpy = "0 0 0"/>
 </joint>
 <!--joints for urf-->
@@ -338,6 +338,6 @@
   <parent link = "link_chassis"/>
   <child link = "urf_limb"/>
-    <origin xyz = "0.5 -0.25 0" rpy = "0 1.57 -0.785"/>
-      <limit lower = "-0.785" upper = "0.785" effort = "10" velocity = "3"/>
+    <origin xyz = "0.5 -0.25 -0.1" rpy = "0 1.57 -0.785"/>
+      <limit lower = "-1.57" upper = "1.57" effort = "10" velocity = "3"/>
       <axis xyz = "1 0 0"/>
 </joint>
@@ -345,5 +345,5 @@
   <parent link = "urf_limb"/>
   <child link = "urf_femur"/>
-    <origin xyz = "0 0 0.25" rpy = "0 1.57 0"/>
+    <origin xyz = "0 0 0.25" rpy = "0 2.355 0"/>
       <limit lower = "-0.785" upper = "0.785" effort = "10" velocity = "3"/>
       <axis xyz = "0 1 0"/>
@@ -352,5 +352,5 @@
   <parent link = "urf_femur"/>
   <child link = "urf_leg"/>
-    <origin xyz = "0 0 -0.25" rpy = "0 1.57 0"/>
+    <origin xyz = "0 0 -0.25" rpy = "0 2.355 0"/>
       <limit lower = "-0.785" upper = "0.785" effort = "10" velocity = "3"/>
       <axis xyz = "0 1 0"/>
@@ -359,5 +359,5 @@
   <parent link = "urf_leg"/>
   <child link = "urf_paw"/>
-    <origin xyz = "0 0 -0.25" rpy = "0 0 0"/>
+    <origin xyz = "0 0 -0.5" rpy = "0 0 0"/>
 </joint>
 <!--joints for blf-->
@@ -365,6 +365,6 @@
   <parent link = "link_chassis"/>
   <child link = "blf_limb"/>
-    <origin xyz = "-0.5 0.25 0" rpy = "0 1.57 2.355"/>
-      <limit lower = "-0.785" upper = "0.785" effort = "10" velocity = "3"/>
+    <origin xyz = "-0.5 0.25 -0.1" rpy = "0 1.57 2.355"/>
+      <limit lower = "-1.57" upper = "1.57" effort = "10" velocity = "3"/>
       <axis xyz = "1 0 0"/>
 </joint>
@@ -372,5 +372,5 @@
   <parent link = "blf_limb"/>
   <child link = "blf_femur"/>
-    <origin xyz = "0 0 0.25" rpy = "0 1.57 0"/>
+    <origin xyz = "0 0 0.25" rpy = "0 2.355 0"/>
       <limit lower = "-0.785" upper = "0.785" effort = "10" velocity = "3"/>
       <axis xyz = "0 1 0"/>
@@ -379,5 +379,5 @@
   <parent link = "blf_femur"/>
   <child link = "blf_leg"/>
-    <origin xyz = "0 0 -0.25" rpy = "0 1.57 0"/>
+    <origin xyz = "0 0 -0.25" rpy = "0 2.355 0"/>
       <limit lower = "-0.785" upper = "0.785" effort = "10" velocity = "3"/>
       <axis xyz = "0 1 0"/>
@@ -386,5 +386,5 @@
   <parent link = "blf_leg"/>
   <child link = "blf_paw"/>
-    <origin xyz = "0 0 -0.25" rpy = "0 0 0"/>
+    <origin xyz = "0 0 -0.5" rpy = "0 0 0"/>
 </joint>
 <!--joints for brf-->
@@ -392,6 +392,6 @@
   <parent link = "link_chassis"/>
   <child link = "brf_limb"/>
-    <origin xyz = "-0.5 -0.25 0" rpy = "0 1.57 3.925"/>
-      <limit lower = "-0.785" upper = "0.785" effort = "10" velocity = "3"/>
+    <origin xyz = "-0.5 -0.25 -0.1" rpy = "0 1.57 3.925"/>
+      <limit lower = "-1.57" upper = "1.57" effort = "10" velocity = "3"/>
       <axis xyz = "1 0 0"/>
 </joint>
@@ -399,5 +399,5 @@
   <parent link = "brf_limb"/>
   <child link = "brf_femur"/>
-    <origin xyz = "0 0 0.25" rpy = "0 1.57 0"/>
+    <origin xyz = "0 0 0.25" rpy = "0 2.355 0"/>
       <limit lower = "-0.785" upper = "0.785" effort = "10" velocity = "3"/>
       <axis xyz = "0 1 0"/>
@@ -406,5 +406,5 @@
   <parent link = "brf_femur"/>
   <child link = "brf_leg"/>
-    <origin xyz = "0 0 -0.25" rpy = "0 1.57 0"/>
+    <origin xyz = "0 0 -0.25" rpy = "0 2.355 0"/>
       <limit lower = "-0.785" upper = "0.785" effort = "10" velocity = "3"/>
       <axis xyz = "0 1 0"/>
@@ -413,5 +413,5 @@
   <parent link = "brf_leg"/>
   <child link = "brf_paw"/>
-    <origin xyz = "0 0 -0.25" rpy = "0 0 0"/>
+    <origin xyz = "0 0 -0.5" rpy = "0 0 0"/>
 </joint>
 </robot>
